File: HALL_Sense.sch (KiCad schematic (older format))
At the start: 36 parts, among them J3 Screw_Terminal_01x03, J4 Screw_Terminal_01x02, U11 74HC14

Commit message: Update_04232021
Changed lines of the file:
@@
 	7250 2300 9100 2300
 Wire Wire Line
-	9000 2750 9000 2200
-Connection ~ 9000 2200
+	10200 2600 10200 4400
 Wire Wire Line
-	9000 2200 10850 2200
+	8300 2200 8900 2200
 Wire Wire Line
-	8300 2200 9000 2200
+	8900 2750 8900 2200
+Connection ~ 8900 2200
 Wire Wire Line
-	8900 2750 8900 2600
+	8900 2200 10850 2200
 Wire Wire Line
-	8900 2600 10200 2600
+	9000 2750 9000 2600
 Wire Wire Line
-	10200 2600 10200 4400
+	9000 2600 10200 2600
 $EndSCHEMATC

Commit message: main
Changed lines of the file:
@@
 $Descr A4 11693 8268
 encoding utf-8
-Sheet 3 7
+Sheet 3 8
 Title ""
 Date ""
@@
 	1    0    0    -1
 $EndComp
-Text GLabel 3750 1250 0    50   Input ~ 0
+Text GLabel 3750 1250 0    50   Output ~ 0
 PB0_HALL_S1
-Text GLabel 3750 2300 0    50   Input ~ 0
+Text GLabel 3750 2300 0    50   Output ~ 0
 PB1_HALL_S2
-Text GLabel 3750 3350 0    50   Input ~ 0
+Text GLabel 3750 3350 0    50   Output ~ 0
 PB2_HALL_S3
 Wire Wire Line
