File: Motor_Driver.sch (KiCad schematic (older format))
At the start: 86 parts, among them J2 Screw_Terminal_01x03, Q1 STB100N10F7, Q2 STB100N10F7, Q3 STB100N10F7, Q4 STB100N10F7, Q5 STB100N10F7, Q6 STB100N10F7, U2 A6387, U3 A6387, U4 A6387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

Commit message: main
Changed lines of the file:
@@
 $Descr A3 16535 11693
 encoding utf-8
-Sheet 2 7
+Sheet 2 8
 Title ""
 Date ""
@@
 Text GLabel 4100 6500 0    50   Input ~ 0
 PA10_TIM1_CH3
-Text GLabel 6800 10450 0    50   Input ~ 0
+Text GLabel 6800 10450 0    50   Output ~ 0
 PC3_ADC2_IN9
-Text GLabel 8600 10450 0    50   Input ~ 0
+Text GLabel 8600 10450 0    50   Output ~ 0
 PA0_ADC2_IN1
-Text GLabel 10450 10450 0    50   Input ~ 0
+Text GLabel 10450 10450 0    50   Output ~ 0
 PA1_ADC2_IN2
-Text GLabel 11800 2800 2    50   Input ~ 0
+Text GLabel 11800 2800 2    50   Output ~ 0
 PC0_ADC1_IN6
-Text GLabel 11800 5250 2    50   Input ~ 0
+Text GLabel 11800 5250 2    50   Output ~ 0
 PC1_ADC1_IN7
-Text GLabel 11800 7700 2    50   Input ~ 0
+Text GLabel 11800 7700 2    50   Output ~ 0
 PC2_ADC1_IN8
 Wire Wire Line
