File: Speed_Brake.sch (KiCad schematic (older format))
At the start: 38 parts, among them J7 Screw_Terminal_01x03, J8 Screw_Terminal_01x02, J9 Screw_Terminal_01x02, U13 MCP6001-OT, U14 MCP6001-OT, U15 MCP6001-OT

Commit message: Update_0426_2021
Parts:
- J9: footprint TerminalBlock_4Ucon:TerminalBlock_4Ucon_1x02_P3.50mm_Vertical -> TerminalBlock_4Ucon:TerminalBlock_4Ucon_1x02_P3.50mm_Horizontal
Changed lines of the file:
@@
 F 0 "J9" H 8218 5267 50  0000 C CNN
 F 1 "Screw_Terminal_01x02" H 8218 5266 50  0001 C CNN
-F 2 "TerminalBlock_4Ucon:TerminalBlock_4Ucon_1x02_P3.50mm_Vertical" H 8300 5500 50  0001 C CNN
+F 2 "TerminalBlock_4Ucon:TerminalBlock_4Ucon_1x02_P3.50mm_Horizontal" H 8300 5500 50  0001 C CNN
 F 3 "~" H 8300 5500 50  0001 C CNN
 	1    8300 5500

Commit message: main
Connections:
- net labels added: BRAKE_L_GND, BRAKE_R_GND, SPEED_ADJ_GND
Changed lines of the file:
@@
 $Descr A4 11693 8268
 encoding utf-8
-Sheet 6 7
+Sheet 6 8
 Title ""
 Date ""
@@
 	1    0    0    -1
 $EndComp
-Text GLabel 2700 1450 0    50   Input ~ 0
+Text GLabel 2700 1450 0    50   Output ~ 0
 PB13_ADC3_IN5
-Text GLabel 3000 3350 0    50   Input ~ 0
+Text GLabel 3000 3350 0    50   Output ~ 0
 PB12_TIM1_BKIN
-Text GLabel 2600 5300 0    50   Input ~ 0
+Text GLabel 2600 5300 0    50   Output ~ 0
 PB11
 Text Label 4300 5600 0    50   ~ 0
@@
 Wire Wire Line
 	3000 3350 3150 3350
+Text Label 7400 3950 0    50   ~ 0
+BRAKE_L_GND
+Text Label 7400 5900 0    50   ~ 0
+BRAKE_R_GND
+Text Label 6800 2050 0    50   ~ 0
+SPEED_ADJ_GND
 $EndSCHEMATC

Commit message: 0429_2021_Update
Connections:
- net labels removed: VSS
Changed lines of the file:
@@
 $EndComp
 Connection ~ 4750 5600
-$Comp
-L power:VSS #PWR?
-U 1 1 60C703B6
-P 4750 5000
-AR Path="/605EBA19/60C703B6" Ref="#PWR?"  Part="1"
-AR Path="/60C0FF99/60C703B6" Ref="#PWR0155"  Part="1"
-F 0 "#PWR0155" H 4750 4850 50  0001 C CNN
-F 1 "VSS" H 4765 5173 50  0000 C CNN
-F 2 "" H 4750 5000 50  0001 C CNN
-F 3 "" H 4750 5000 50  0001 C CNN
-	1    4750 5000
-	1    0    0    -1
-$EndComp
 Wire Wire Line
 	5400 5200 5400 4700
@@
 Text Label 6800 2050 0    50   ~ 0
 SPEED_ADJ_GND
+$Comp
+L power:GND #PWR?
+U 1 1 608A6683
+P 4750 5000
+AR Path="/605EBA19/608A6683" Ref="#PWR?"  Part="1"
+AR Path="/60C0FF99/608A6683" Ref="#PWR0155"  Part="1"
+F 0 "#PWR0155" H 4750 4750 50  0001 C CNN
+F 1 "GND" H 4755 4827 50  0000 C CNN
+F 2 "" H 4750 5000 50  0001 C CNN
+F 3 "" H 4750 5000 50  0001 C CNN
+	1    4750 5000
+	-1   0    0    1
+$EndComp
 $EndSCHEMATC
