File: BLDC_Tester_Board.kicad_pcb (KiCad board)
At the start: 2 copper layers, 227 parts, among them J1 nucleo-g474re, J10 Screw_Terminal_01x02, J2 Screw_Terminal_01x03, J3 Screw_Terminal_01x03, J4 Screw_Terminal_01x02, J5 Screw_Terminal_01x02, J6 Screw_Terminal_01x02, J7 Screw_Terminal_01x03, J8 Screw_Terminal_01x02, J9 Screw_Terminal_01x02, Q1 STB100N10F7, Q2 STB100N10F7, Q3 STB100N10F7, Q4 STB100N10F7, Q5 STB100N10F7, Q6 STB100N10F7, U1 MCP6001-OT, U11 74HC14, U12 74HC14, U13 MCP6001-OT, U14 MCP6001-OT, U15 MCP6001-OT, U16 L4971, U17 LM1117-5.0, U18 LM1117-3.3, U2 A6387, U3 A6387, U4 A6387, U5 TSC2012IDT, U6 TSC2012IDT, U7 TSC2012IDT

Commit message: Update_04232021
Parts:
- moved J6 299.5 mm to (430.3, 311.0), turned to 90 degrees
- moved C31 293.3 mm to (419.2, 307.8), turned to 270 degrees
- moved TP24 290.9 mm to (346.7, 299.3)
- moved R49 289.6 mm to (356.7, 297.7)
- moved R50 284.8 mm to (351.9, 294.4), turned to 180 degrees
- moved C29 283.4 mm to (392.6, 302.9), turned to 270 degrees
- moved TP22 280.2 mm to (412.2, 298.6)
- moved U12 278.7 mm to (377.2, 294.8)
- moved J5 277.6 mm to (428.2, 297.8), turned to 90 degrees
- moved D14 277.1 mm to (363.0, 299.3), turned to 180 degrees
- moved R55 276.4 mm to (395.6, 293.5), turned to 180 degrees
- moved D16 275.6 mm to (401.7, 302.9), turned to 90 degrees
- moved FB7 275.5 mm to (395.6, 302.9), turned to 180 degrees
- moved R56 274.6 mm to (368.3, 297.7), turned to 180 degrees
- moved C30 271.5 mm to (389.5, 302.9), turned to 270 degrees
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Connections:
- C29 pad 2: /Speed_Sense/ENCODER_GND -> GND
- C30 pad 2: /Speed_Sense/ENCODER_GND -> GND
- D13 pad 1: /HALL_Sense/HALL_5V -> /HALL_Sense/HALL_S1
- D13 pad 3: /HALL_Sense/HALL_S1 -> /HALL_Sense/HALL_5V
- D16 pad 1: /Speed_Sense/ENCODER_B_IN -> /Speed_Sense/ENCODER_5V
- D16 pad 3: /Speed_Sense/ENCODER_A_IN -> Net-(D16-Pad3)
- D16 pad 4: Net-(D16-Pad4) -> /Speed_Sense/ENCODER_A_IN
- D16 pad 6: /Speed_Sense/ENCODER_5V -> /Speed_Sense/ENCODER_B_IN
- U12 pad 1: Net-(C29-Pad1) -> Net-(U12-Pad1)
- U12 pad 10: (no net) -> Net-(R50-Pad1)
- U12 pad 11: (no net) -> Net-(C30-Pad1)
- U12 pad 12: (no net) -> Net-(U12-Pad12)
- U12 pad 13: (no net) -> Net-(U12-Pad13)
- U12 pad 2: Net-(R48-Pad1) -> Net-(U12-Pad2)
- U12 pad 4: Net-(R50-Pad1) -> Net-(R57-Pad1)
- U12 pad 8: Net-(R57-Pad1) -> Net-(R48-Pad1)
- U12 pad 9: Net-(C30-Pad1) -> Net-(C29-Pad1)
Routing:
- net /DC to DC/3V3: track 0.00 -> 78.8 mm
- net /DC to DC/5V: track 0.00 -> 42.5 mm
- net Net-(C24-Pad1): track 0.00 -> 37.5 mm, vias 0 -> 2
- net Net-(C26-Pad1): track 0.00 -> 37.5 mm, vias 0 -> 2
- net Net-(C25-Pad1): track 0.00 -> 37.0 mm, vias 0 -> 3
- net Net-(R35-Pad1): track 0.00 -> 35.2 mm, vias 0 -> 2
- net Net-(R37-Pad1): track 0.00 -> 34.5 mm, vias 0 -> 2
- net Net-(R33-Pad1): track 0.00 -> 33.5 mm, vias 0 -> 2
- net Net-(C30-Pad1): track 0.00 -> 32.6 mm, vias 0 -> 2
- net Net-(C29-Pad1): track 0.00 -> 32.6 mm, vias 0 -> 2
- net /HALL_Sense/HALL_S3: track 0.00 -> 29.4 mm, vias 0 -> 2
- net Net-(C48-Pad1): track 0.00 -> 27.2 mm
- net Net-(C45-Pad1): track 0.00 -> 26.7 mm
- net /DC to DC/10V: track 0.00 -> 25.1 mm
- net /HALL_Sense/HALL_S2: track 0.00 -> 24.5 mm, vias 0 -> 2
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
Commit message: Update_0426_2021
Parts:
- J9: footprint TerminalBlock_4Ucon:TerminalBlock_4Ucon_1x02_P3.50mm_Vertical -> TerminalBlock_4Ucon:TerminalBlock_4Ucon_1x02_P3.50mm_Horizontal
- moved J10 292.8 mm to (457.8, 278.8), turned to 90 degrees
- moved FL1 286.7 mm to (439.3, 284.8), turned to 180 degrees
- moved C2 256.0 mm to (307.8, 265.8)
- moved C3 256.0 mm to (316.5, 265.8)
- moved FB2 256.0 mm to (312.2, 265.8)
- moved F1 253.1 mm to (420.9, 262.5)
- moved TP20 190.5 mm to (405.1, 130.9)
- moved TP21 178.4 mm to (398.9, 130.8)
- moved FB6 175.1 mm to (426.1, 133.5), turned to 180 degrees
- moved C31 161.2 mm to (446.4, 148.9)
- moved J6 161.0 mm to (457.8, 152.4)
- moved TP17 159.8 mm to (436.8, 122.2)
- moved C27 159.3 mm to (446.4, 128.3)
- moved J4 158.4 mm to (457.8, 131.8)
- moved C23 158.1 mm to (410.2, 110.3)
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Routing:
- net /Speed_Sense/ENCODER_5V: track 0.00 -> 63.7 mm, vias 0 -> 4
- net /MotorDriver/MOT_PV: track 7.71 -> 44.8 mm
- net /MotorDriver/ISEN_PV: track 0.00 -> 26.3 mm
- net /MotorDriver/ISEN_PU: track 0.00 -> 26.3 mm
- net /MotorDriver/ISEN_PW: track 0.00 -> 26.2 mm
- net /HALL_Sense/HALL_S1: track 17.0 -> 40.4 mm
- net Net-(C43-Pad1): track 22.7 -> 0.00 mm
- net /DC to DC/10V: track 25.1 -> 44.5 mm
- net /Speed_Sense/ENCODER_B_IN: track 18.7 -> 34.2 mm
- net /Speed_Sense/ENCODER_A_IN: track 23.8 -> 39.2 mm
- net /HALL_Sense/HALL_S2: track 24.5 -> 39.6 mm
- net /HALL_Sense/HALL_S3: track 29.4 -> 43.5 mm
- net Net-(C9-Pad1): track 11.9 -> 25.2 mm
- net Net-(C48-Pad1): track 27.2 -> 13.8 mm
- net Net-(C7-Pad1): track 11.9 -> 25.2 mm
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- added copper zone on F.Cu, net /MotorDriver/ISEN_PU
- added copper zone on F.Cu, net /MotorDriver/ISEN_PV
- added copper zone on F.Cu, net /MotorDriver/ISEN_PW
- added copper zone on F.Cu, net /MotorDriver/MOT_PU
- added copper zone on F.Cu, net /MotorDriver/MOT_PV
- added copper zone on F.Cu, net /MotorDriver/MOT_PW

Commit message: main
Parts:
- added C4: 100uF/35V, Capacitor_THT:CP_Radial_D6.3mm_P2.50mm, F.Cu at (336.0, 284.7)
- added C53: 100nF, Capacitor_SMD:C_0603_1608Metric_Pad1.08x0.95mm_HandSolder, F.Cu at (307.3, 124.5)
- added C54: 100nF, Capacitor_SMD:C_0603_1608Metric_Pad1.08x0.95mm_HandSolder, F.Cu at (308.2, 145.4)
- added C55: 100nF, Capacitor_SMD:C_0603_1608Metric_Pad1.08x0.95mm_HandSolder, F.Cu at (315.6, 154.7)
- added C56: 100nF, Capacitor_SMD:C_0603_1608Metric_Pad1.08x0.95mm_HandSolder, F.Cu at (300.4, 154.7)
- added C57: 100nF, Capacitor_SMD:C_0603_1608Metric_Pad1.08x0.95mm_HandSolder, F.Cu at (300.4, 159.8)
- added C58: 100nF, Capacitor_SMD:C_0603_1608Metric_Pad1.08x0.95mm_HandSolder, F.Cu at (308.2, 150.6)
- added C59: 100nF, Capacitor_SMD:C_0603_1608Metric_Pad1.08x0.95mm_HandSolder, F.Cu at (308.2, 166.8)
- added D21: PESD2CAN, Package_TO_SOT_SMD:SOT-23, F.Cu at (295.9, 126.6)
- added D22: D_TVS_x2_AAC, Package_TO_SOT_SMD:SOT-23, F.Cu at (295.9, 149.5)
- added D23: SM712_SOT23, Package_TO_SOT_SMD:SOT-23, F.Cu at (295.9, 170.8)
- added FB15: Ferrite_Bead, Resistor_SMD:R_0603_1608Metric_Pad0.98x0.95mm_HandSolder, F.Cu at (300.4, 127.6)
- added FB16: Ferrite_Bead, Resistor_SMD:R_0603_1608Metric_Pad0.98x0.95mm_HandSolder, F.Cu at (300.4, 150.6)
- added FB17: Ferrite_Bead, Resistor_SMD:R_0603_1608Metric_Pad0.98x0.95mm_HandSolder, F.Cu at (300.4, 171.8)
- added J11: Screw_Terminal_01x03, TerminalBlock_4Ucon:TerminalBlock_4Ucon_1x03_P3.50mm_Horizontal, F.Cu at (291.8, 113.5)
- added J12: Screw_Terminal_01x03, TerminalBlock_4Ucon:TerminalBlock_4Ucon_1x03_P3.50mm_Horizontal, F.Cu at (292.0, 136.3)
- added J13: Screw_Terminal_01x03, TerminalBlock_4Ucon:TerminalBlock_4Ucon_1x03_P3.50mm_Horizontal, F.Cu at (292.0, 157.5)
- added JP2: Jumper_3_Bridged12, Connector_PinHeader_2.54mm:PinHeader_1x03_P2.54mm_Vertical, F.Cu at (320.0, 169.5)
- added JP3: Jumper_NC_Small, Connector_PinHeader_2.54mm:PinHeader_1x02_P2.54mm_Vertical, F.Cu at (300.4, 117.2)
- added JP4: Jumper_NC_Small, Connector_PinHeader_2.54mm:PinHeader_1x02_P2.54mm_Vertical, F.Cu at (300.4, 138.2)
- added JP5: Jumper_3_Bridged12, Connector_PinHeader_2.54mm:PinHeader_1x03_P2.54mm_Vertical, F.Cu at (320.0, 158.1)
- added R71: 120, Resistor_SMD:R_0805_2012Metric_Pad1.20x1.40mm_HandSolder, F.Cu at (300.4, 122.6)
- added R72: 220, Resistor_SMD:R_0805_2012Metric_Pad1.20x1.40mm_HandSolder, F.Cu at (300.4, 143.4)
- added U19: MCP2558FD-xSN, Package_SO:SOIC-8_3.9x4.9mm_P1.27mm, F.Cu at (308.0, 118.7)
- added U20: MAX485E, Package_SO:SOP-8_3.9x4.9mm_P1.27mm, F.Cu at (308.2, 139.7)
- added U21: MAX3232, Package_SO:SO-16_3.9x9.9mm_P1.27mm, F.Cu at (308.2, 159.2)
- moved TP34 33.5 mm to (343.4, 144.2)
- moved C34 16.7 mm to (336.8, 134.9)
- moved R68 15.0 mm to (324.9, 136.6)
- moved C32 14.8 mm to (335.0, 124.5)
- moved D17 14.8 mm to (330.2, 121.0)
- moved FB10 14.8 mm to (335.0, 121.0)
- moved FB9 14.8 mm to (330.2, 124.5)
- moved J7 14.8 mm to (333.7, 114.7)
- moved R58 14.8 mm to (330.2, 127.6)
- moved U13 14.8 mm to (330.2, 133.6)
- moved TP32 14.2 mm to (324.9, 144.2)
- moved FB8 11.2 mm to (319.3, 127.6)
- moved C41 9.99 mm to (320.2, 121.0)
- moved J1 8.69 mm to (327.1, 213.4)
- moved R59 5.60 mm to (324.9, 124.5), turned to 0 degrees
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Connections:
- net Net-(C41-Pad2) renamed /Speed control and Brake/SPEED_ADJ_GND
- net Net-(D18-Pad2) renamed /Speed control and Brake/BRAKE_L_GND
- net Net-(D19-Pad2) renamed /Speed control and Brake/BRAKE_R_GND
- J1 pad L21: Net-(J1-PadL21) -> PB7
- J1 pad L4: Net-(J1-PadL4) -> PD2_UART5_RX
- J1 pad R17: Net-(J1-PadR17) -> PB6_CAN2_TX
- J1 pad R27: Net-(J1-PadR27) -> PB4_UART5_DE
- J1 pad R29: Net-(J1-PadR29) -> PB5_CAN2_RX
Routing:
- net PC8_TIM3_CH3: track 0.00 -> 109.9 mm, vias 0 -> 1
- net PC9_TIM3_CH4: track 0.00 -> 107.8 mm, vias 0 -> 1
- net PB2_HALL_S3: track 6.42 -> 109.9 mm, vias 0 -> 3
- net PB12_TIM1_BKIN: track 0.00 -> 67.7 mm, vias 0 -> 1
- net PB11: track 0.00 -> 49.7 mm, vias 0 -> 1
- net /DC to DC/5V: track 29.3 -> 69.4 mm, vias 0 -> 2
- net /RS485 & CANFD interface/RS485-: track 0.00 -> 33.1 mm, vias 0 -> 1
- net PB1_HALL_S2: track 4.29 -> 37.1 mm
- net /RS485 & CANFD interface/L485_RX: track 0.00 -> 31.7 mm, vias 0 -> 1
- net /RS485 & CANFD interface/CAN-: track 0.00 -> 29.5 mm, vias 0 -> 1
- net /RS485 & CANFD interface/RS232_TX: track 0.00 -> 25.5 mm, vias 0 -> 1
- net /RS485 & CANFD interface/L485_TX: track 0.00 -> 24.4 mm, vias 0 -> 1
- net /RS485 & CANFD interface/RS485+: track 0.00 -> 23.0 mm
- net /RS485 & CANFD interface/CAN+: track 0.00 -> 22.6 mm
- net Net-(R69-Pad1): track 0.00 -> 22.0 mm, vias 0 -> 3
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
Commit message: 0428_2021_Update
Parts:
- removed the C4 at (336.0, 284.7)
- F1: footprint Fuse:Fuse_SunFuse-6HP -> Fuse:Fuseholder_Cylinder-5x20mm_Stelvio-Kontek_PTF78_Horizontal_Open
- FL1: footprint Inductor_THT:Choke_Schaffner_RN102-04-14.0x14.0mm -> Inductor_THT:Choke_Schaffner_RN242-04-18.0x31.0mm
- J1: value nucleo-g474re -> stm32-nucleo64-Morpho; footprint STM32-Nucleo-Board:stm32-nucleo64-board -> STM32-Nucleo-Board:stm32-nucleo64-Morpho
- moved FB3 84.9 mm to (325.2, 188.0), turned to 270 degrees
- moved FB1 69.3 mm to (326.5, 238.7), turned to 90 degrees
- moved RV1 51.6 mm to (325.0, 258.3), turned to 90 degrees
- moved C4 50.8 mm to (320.0, 231.1)
- moved TP28 45.5 mm to (287.5, 260.3)
- moved C51 43.5 mm to (314.0, 266.6)
- moved R1 41.0 mm to (315.5, 252.3), turned to 270 degrees
- moved L1 40.8 mm to (341.9, 263.3), turned to 90 degrees
- moved C49 40.7 mm to (334.3, 256.0), turned to 180 degrees
- moved TP27 37.0 mm to (314.0, 273.0)
- moved U18 36.6 mm to (305.3, 263.5), turned to 90 degrees
- moved U17 35.0 mm to (323.2, 266.6), turned to 180 degrees
- moved JP1 35.0 mm to (296.5, 251.4), turned to 270 degrees
- moved C52 34.6 mm to (297.2, 260.3), turned to 270 degrees
- moved D20 34.0 mm to (348.9, 268.9), turned to 270 degrees
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Connections:
- J10 pad 1: Net-(F1-Pad2) -> Net-(FL1-Pad1)
- J10 pad 2: Net-(FL1-Pad1) -> Net-(F1-Pad2)
Routing:
- net PB7: track 0.00 -> 167.6 mm, vias 0 -> 2
- net PB0_HALL_S1: track 6.42 -> 143.0 mm, vias 0 -> 2
- net PB5_CAN2_RX: track 0.00 -> 134.0 mm, vias 0 -> 3
- net PB4_UART5_DE: track 0.00 -> 114.1 mm, vias 0 -> 3
- net PB6_CAN2_TX: track 0.00 -> 111.3 mm, vias 0 -> 3
- net /DC to DC/5V: track 69.4 -> 167.5 mm, vias 2 -> 3
- net Net-(FB3-Pad2): track 0.00 -> 97.9 mm, vias 0 -> 1
- net PA11_TIM1_CH1N: track 10.8 -> 104.7 mm, vias 0 -> 1
- net PA1_ADC2_IN2: track 15.7 -> 102.6 mm, vias 0 -> 3
- net PA8_TIM1_CH1: track 10.8 -> 96.8 mm, vias 0 -> 1
- net PC2_ADC1_IN8: track 0.00 -> 80.1 mm, vias 0 -> 2
- net PB13_ADC3_IN5: track 0.00 -> 76.7 mm, vias 0 -> 3
- net PB1_HALL_S2: track 37.1 -> 99.2 mm, vias 0 -> 3
- net PA12_TIM1_CH2N: track 10.8 -> 71.3 mm, vias 0 -> 1
- net PA0_ADC2_IN1: track 15.7 -> 68.9 mm, vias 0 -> 1
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Other:
- board outline added: 183.5 x 182.2 mm

Commit message: 0429_2021_Update
Parts:
- moved TP20 56.3 mm to (361.1, 166.1)
- moved FB1 30.1 mm to (300.5, 254.0), turned to 0 degrees
- moved C4 26.1 mm to (307.4, 254.0), turned to 180 degrees
- moved TP21 24.3 mm to (412.2, 151.1)
- moved FB4 22.4 mm to (426.1, 111.3)
- moved FB2 18.8 mm to (311.8, 254.0), turned to 180 degrees
- moved C15 15.7 mm to (386.5, 260.4), turned to 90 degrees
- moved C19 15.5 mm to (386.5, 187.1), turned to 90 degrees
- moved C17 15.4 mm to (386.5, 223.4), turned to 90 degrees
- moved C20 13.9 mm to (389.5, 232.2), turned to 0 degrees
- moved C22 13.4 mm to (389.5, 159.7), turned to 0 degrees
- moved C21 13.3 mm to (389.5, 196.3), turned to 0 degrees
- moved TP28 9.46 mm to (284.2, 269.2)
- moved C2 8.32 mm to (312.1, 265.7)
- moved C44 8.32 mm to (366.7, 266.5)
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Connections:
- J1 pad L3: Net-(J1-PadL3) -> PC12_UART5_TX
- U15 pad 2: VSS -> GND
Routing:
- net /DC to DC/3V3: track 99.7 -> 521.1 mm, vias 0 -> 18
- net /DC to DC/5V: track 167.5 -> 371.5 mm, vias 3 -> 13
- net PC12_UART5_TX: track 0.00 -> 139.8 mm, vias 0 -> 4
- net /DC to DC/10V: track 27.0 -> 141.8 mm, vias 0 -> 7
- net PD2_UART5_RX: track 0.00 -> 108.6 mm, vias 0 -> 5
- net /HALL_Sense/HALL_5V: track 11.4 -> 55.3 mm, vias 0 -> 2
- net /Speed_Sense/ENCODER_GND: track 0.00 -> 39.0 mm
- net /HALL_Sense/HALL_GND: track 0.00 -> 37.3 mm
- net PC1_ADC1_IN7: track 36.4 -> 65.5 mm
- net PC2_ADC1_IN8: track 80.1 -> 109.2 mm
- net PC3_ADC2_IN9: track 15.7 -> 37.6 mm, vias 0 -> 2
- net PC0_ADC1_IN6: track 38.1 -> 59.7 mm
- net /MotorDriver/MOT_PU: track 8.86 -> 28.4 mm
- net PA12_TIM1_CH2N: track 71.3 -> 83.1 mm, vias 1 -> 3
- net GND: track 0.00 -> 11.8 mm
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
Commit message: 0503_2021_Update
Parts:
- added C63: 4.7nF, Capacitor_SMD:C_0603_1608Metric_Pad1.08x0.95mm_HandSolder, F.Cu at (350.8, 268.4)
- added C64: 120nF, Capacitor_SMD:C_0603_1608Metric_Pad1.08x0.95mm_HandSolder, F.Cu at (368.7, 268.4)
- added C65: 680nF, Capacitor_SMD:C_0603_1608Metric_Pad1.08x0.95mm_HandSolder, F.Cu at (364.4, 271.5)
- added R73: 750, Resistor_SMD:R_0603_1608Metric_Pad0.98x0.95mm_HandSolder, F.Cu at (359.9, 268.4)
- added R74: 430, Resistor_SMD:R_0603_1608Metric_Pad0.98x0.95mm_HandSolder, F.Cu at (355.4, 268.4)
- added R75: 1K, Resistor_SMD:R_0603_1608Metric_Pad0.98x0.95mm_HandSolder, F.Cu at (364.4, 268.4)
- C44: value 22nF -> 1000nF
- C45: value 100nF -> 1000nF
- C46: value 100nF -> 68nF
- C47: value 2.7nF -> 100nF
- C48: value 10pF -> 1000nF
- L1: value 220uH -> 33uH
- R64: value 9.1K -> 0
- R65: value 20K -> 51.1K
- R66: value 2.7K -> 36K; footprint Resistor_SMD:R_1206_3216Metric_Pad1.30x1.75mm_HandSolder -> Resistor_SMD:R_0603_1608Metric_Pad0.98x0.95mm_HandSolder
- R67: footprint Resistor_SMD:R_1206_3216Metric_Pad1.30x1.75mm_HandSolder -> Resistor_SMD:R_0603_1608Metric_Pad0.98x0.95mm_HandSolder
- U16: value L4971 -> L7987; footprint Package_DIP:DIP-8_W7.62mm_LongPads -> Package_SO:HTSSOP-16-1EP_4.4x5mm_P0.65mm_EP3x3mm
- moved FB3 65.7 mm to (294.6, 246.1)
- moved C48 30.3 mm to (372.4, 283.3), turned to 180 degrees
- moved C46 26.7 mm to (375.6, 271.8), turned to 90 degrees
- moved C45 23.8 mm to (379.6, 271.8), turned to 270 degrees
- moved C44 19.7 mm to (382.6, 278.2), turned to 90 degrees
- moved U16 19.6 mm to (370.4, 278.1), turned to 180 degrees
- moved R66 19.4 mm to (359.9, 274.5), turned to 180 degrees
- moved U1 18.9 mm to (288.7, 263.9), turned to 180 degrees
- moved C1 18.5 mm to (293.7, 258.4)
- moved R1 18.5 mm to (297.2, 258.5)
- moved C2 18.5 mm to (293.7, 263.8)
- moved R2 18.5 mm to (297.2, 263.8)
- moved RV1 17.7 mm to (307.3, 264.7)
- moved C49 16.9 mm to (342.5, 279.1), turned to 90 degrees
- moved R64 15.5 mm to (379.6, 278.1), turned to 270 degrees
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Connections:
- C44 pad 1: Net-(C44-Pad1) -> Net-(C43-Pad1)
- C45 pad 1: Net-(C45-Pad1) -> GND
- C47 pad 2: GND -> Net-(C47-Pad2)
- C48 pad 1: Net-(C48-Pad1) -> /DC to DC/10V
- D20 pad 1: Net-(C45-Pad1) -> Net-(C47-Pad1)
- L1 pad 1: Net-(C45-Pad1) -> Net-(C47-Pad1)
- R64 pad 1: Net-(C44-Pad1) -> Net-(C45-Pad2)
- R64 pad 2: Net-(R64-Pad2) -> Net-(C43-Pad1)
- R65 pad 1: Net-(C43-Pad1) -> Net-(R65-Pad1)
- R65 pad 2: Net-(C47-Pad1) -> GND
- R66 pad 1: /DC to DC/10V -> Net-(R66-Pad1)
- R66 pad 2: Net-(C48-Pad1) -> GND
- R67 pad 1: Net-(C48-Pad1) -> /DC to DC/10V
- R67 pad 2: GND -> Net-(C65-Pad2)
- U16 pad 1: GND -> /DC to DC/10V
- U16 pad 2: Net-(C46-Pad1) -> Net-(C43-Pad1)
- U16 pad 3: Net-(C47-Pad1) -> Net-(C43-Pad1)
- U16 pad 4: Net-(C45-Pad1) -> Net-(C45-Pad2)
- U16 pad 5: Net-(C43-Pad1) -> Net-(C45-Pad2)
- U16 pad 6: Net-(C45-Pad2) -> Net-(C46-Pad1)
- U16 pad 7: Net-(R64-Pad2) -> Net-(U16-Pad7)
- U16 pad 8: Net-(C48-Pad1) -> Net-(C64-Pad2)
Routing:
- net /DC to DC/10V: track 141.8 -> 299.1 mm, vias 7 -> 10
- net /DC to DC/3V3: track 521.1 -> 657.5 mm, vias 18 -> 21
- net /MCU/VREF+: track 2.90 -> 101.9 mm, vias 0 -> 2
- net Net-(FB3-Pad2): track 97.9 -> 4.36 mm, vias 1 -> 0
- net /MCU/VDD: track 6.85 -> 59.8 mm, vias 0 -> 1
- net Net-(C65-Pad2): track 0.00 -> 29.2 mm
- net /MCU/DC5V_IN: track 0.00 -> 28.9 mm, vias 0 -> 2
- net /DC to DC/5V: track 371.5 -> 399.3 mm
- net VSS: track 0.00 -> 25.0 mm, vias 0 -> 2
- net Net-(C48-Pad1): track 23.1 -> 0.00 mm
- net Net-(C45-Pad1): track 22.2 -> 0.00 mm, vias 1 -> 0
- net Net-(C64-Pad2): track 0.00 -> 18.0 mm
- net Net-(C43-Pad1): track 4.01 -> 17.0 mm
- net Net-(R65-Pad1): track 0.00 -> 11.0 mm
- net Net-(R66-Pad1): track 0.00 -> 8.41 mm
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